File: pcb/M,S/Flake.kicad_sch (KiCad schematic)
At the start: 50 parts, among them SW1 SW_Push, SW10 SW_Push, SW11 SW_Push, SW12 SW_Push, SW13 SW_Push, SW14 SW_Push, SW15 SW_Push, SW16 SW_Push, SW17 SW_Push, SW18 SW_Push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

Commit message: feat(enclosure): no chamfer version for easier print
Parts:
- SW1, SW10, SW11, SW12, SW13, SW14, SW15, SW16, SW17, SW18, SW19, SW2, SW20, SW21, SW22, SW23, SW3, SW4, SW5, SW6, SW7, SW8, SW9: footprint axseem:SW_MX_Choc_Hotswap_Reversible -> axseem:SW_MX_Choc_Hotswap_Plated
Changed lines of the file:
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@@
 			)
 		)
-		(property "Footprint" "axseem:SW_MX_Choc_Hotswap_Reversible"
+		(property "Footprint" "axseem:SW_MX_Choc_Hotswap_Plated"
 			(at 38.1 31.75 0)
 			(effects
@@
 			)
 		)
-		(property "Footprint" "axseem:SW_MX_Choc_Hotswap_Reversible"
+		(property "Footprint" "axseem:SW_MX_Choc_Hotswap_Plated"
 			(at 52.07 31.75 0)
 			(effects
@@
 			)
 		)
-		(property "Footprint" "axseem:SW_MX_Choc_Hotswap_Reversible"
+		(property "Footprint" "axseem:SW_MX_Choc_Hotswap_Plated"
 			(at 66.04 57.15 0)
 			(effects
@@
 			)
 		)
-		(property "Footprint" "axseem:SW_MX_Choc_Hotswap_Reversible"
+		(property "Footprint" "axseem:SW_MX_Choc_Hotswap_Plated"
 			(at 107.95 44.45 0)
 			(effects
@@
 			)
 		)
-		(property "Footprint" "axseem:SW_MX_Choc_Hotswap_Reversible"
+		(property "Footprint" "axseem:SW_MX_Choc_Hotswap_Plated"
 			(at 107.95 69.85 0)
 			(effects
@@
 			)
 		)
-		(property "Footprint" "axseem:SW_MX_Choc_Hotswap_Reversible"
+		(property "Footprint" "axseem:SW_MX_Choc_Hotswap_Plated"
 			(at 52.07 69.85 0)
 			(effects
@@
 			)
 		)
-		(property "Footprint" "axseem:SW_MX_Choc_Hotswap_Reversible"
+		(property "Footprint" "axseem:SW_MX_Choc_Hotswap_Plated"
 			(at 66.04 44.45 0)
 			(effects
@@
 			)
 		)
-		(property "Footprint" "axseem:SW_MX_Choc_Hotswap_Reversible"
+		(property "Footprint" "axseem:SW_MX_Choc_Hotswap_Plated"
 			(at 52.07 44.45 0)
 			(effects
@@
 			)
 		)
-		(property "Footprint" "axseem:SW_MX_Choc_Hotswap_Reversible"
+		(property "Footprint" "axseem:SW_MX_Choc_Hotswap_Plated"
 			(at 66.04 31.75 0)
 			(effects
@@
 			)
 		)
-		(property "Footprint" "axseem:SW_MX_Choc_Hotswap_Reversible"
+		(property "Footprint" "axseem:SW_MX_Choc_Hotswap_Plated"
 			(at 38.1 44.45 0)
 			(effects
@@
 			)
 		)
-		(property "Footprint" "axseem:SW_MX_Choc_Hotswap_Reversible"
+		(property "Footprint" "axseem:SW_MX_Choc_Hotswap_Plated"
 			(at 52.07 57.15 0)
 			(effects
@@
 			)
 		)
-		(property "Footprint" "axseem:SW_MX_Choc_Hotswap_Reversible"
+		(property "Footprint" "axseem:SW_MX_Choc_Hotswap_Plated"
 			(at 93.98 31.75 0)
 			(effects
@@
 			)
 		)
-		(property "Footprint" "axseem:SW_MX_Choc_Hotswap_Reversible"
+		(property "Footprint" "axseem:SW_MX_Choc_Hotswap_Plated"
 			(at 80.01 31.75 0)
 			(effects
@@
 			)
 		)
-		(property "Footprint" "axseem:SW_MX_Choc_Hotswap_Reversible"
+		(property "Footprint" "axseem:SW_MX_Choc_Hotswap_Plated"
 			(at 107.95 57.15 0)
 			(effects
@@
 			)
 		)
-		(property "Footprint" "axseem:SW_MX_Choc_Hotswap_Reversible"
+		(property "Footprint" "axseem:SW_MX_Choc_Hotswap_Plated"
 			(at 80.01 69.85 0)
 			(effects
@@
 			)
 		)
-		(property "Footprint" "axseem:SW_MX_Choc_Hotswap_Reversible"
+		(property "Footprint" "axseem:SW_MX_Choc_Hotswap_Plated"
 			(at 80.01 44.45 0)
 			(effects
@@
 			)
 		)
-		(property "Footprint" "axseem:SW_MX_Choc_Hotswap_Reversible"
+		(property "Footprint" "axseem:SW_MX_Choc_Hotswap_Plated"
 			(at 93.98 44.45 0)
 			(effects
@@
 			)
 		)
-		(property "Footprint" "axseem:SW_MX_Choc_Hotswap_Reversible"
+		(property "Footprint" "axseem:SW_MX_Choc_Hotswap_Plated"
 			(at 80.01 57.15 0)
 			(effects
@@
 			)
 		)
-		(property "Footprint" "axseem:SW_MX_Choc_Hotswap_Reversible"
+		(property "Footprint" "axseem:SW_MX_Choc_Hotswap_Plated"
 			(at 38.1 57.15 0)
 			(effects
@@
 			)
 		)
-		(property "Footprint" "axseem:SW_MX_Choc_Hotswap_Reversible"
+		(property "Footprint" "axseem:SW_MX_Choc_Hotswap_Plated"
 			(at 107.95 31.75 0)
 			(effects
@@
 			)
 		)
-		(property "Footprint" "axseem:SW_MX_Choc_Hotswap_Reversible"
+		(property "Footprint" "axseem:SW_MX_Choc_Hotswap_Plated"
 			(at 93.98 69.85 0)
 			(effects
@@
 			)
 		)
-		(property "Footprint" "axseem:SW_MX_Choc_Hotswap_Reversible"
+		(property "Footprint" "axseem:SW_MX_Choc_Hotswap_Plated"
 			(at 93.98 57.15 0)
 			(effects
@@
 			)
 		)
-		(property "Footprint" "axseem:SW_MX_Choc_Hotswap_Reversible"
+		(property "Footprint" "axseem:SW_MX_Choc_Hotswap_Plated"
 			(at 66.04 69.85 0)
 			(effects
